Commit message: param fix

File: husky_description/urdf/accessories/sensor_arch.urdf.xacro (robot description, xacro)
@@ -33,5 +33,5 @@
              <child link="${prefix}sensor_arch_mount_link"/>
 		 <axis xyz="0 0 1"/>
-		 <limit effort="30" velocity="1.0" lower="${-M_PI/2}" upper="${M_PI/2}" />
+		 <limit effort="50" velocity="10.0" lower="${-M_PI/2}" upper="${M_PI/2}" />
 		 <dynamics damping="0.0" friction="0.0"/>
         </joint>

Commit message: simple algorithm implement

File: husky_description/urdf/accessories/sensor_arch.urdf.xacro (robot description, xacro)
@@ -45,13 +45,10 @@
 		</joint>
 	</transmission>
-	<!--gazebo>
-		<plugin name="object_controller" filename="libgazebo_ros_planar_move.so">
-			<commandTopic>cmd_kinect</commandTopic>
-			<odometryTopic>odom</odometryTopic>
-			<odometryFrame>odom</odometryFrame>
-			<odometryRate>20.0</odometryRate>
-			<robotBaseFrame>${prefix}sensor_arch_mount_link</robotBaseFrame>
-		</plugin>
-	</gazebo-->
+	<link name="${prefix}camera_mount"/>
+	<joint name="${prefix}camera_mount_joint" type="fixed">
+	     <xacro:insert_block name="origin"/>
+	     <parent link="${parent}"/>
+	     <child link="${prefix}camera_mount"/>
+	</joint>
     </xacro:macro>
 </robot>

File: husky_description/urdf/husky.urdf.xacro (robot description, xacro)
@@ -27,5 +27,5 @@
   <xacro:arg name="kinect_enabled" default="false" />
   <xacro:arg name="kinect_xyz" default="$(optenv HUSKY_KINECT_XYZ 0 0 0)" />
-  <xacro:arg name="kinect_rpy" default="$(optenv HUSKY_KINECT_RPY 0 0.18 3.14)" />
+  <xacro:arg name="kinect_rpy" default="$(optenv HUSKY_KINECT_RPY 0 0.18 0)" />
   <xacro:property name="husky_front_bumper_extend" value="$(optenv HUSKY_FRONT_BUMPER_EXTEND 0)" />
   <xacro:property name="husky_rear_bumper_extend" value="$(optenv HUSKY_REAR_BUMPER_EXTEND 0)" />
@@ -126,5 +126,5 @@
   <xacro:if value="$(arg kinect_enabled)">
     <xacro:sensor_arch prefix="" parent="top_plate_link">
-      <origin xyz="-0.30 0 0.51" rpy="0 0 -3.14"/>
+      <origin xyz="0 0 0.51" rpy="0 0 0"/>
     </xacro:sensor_arch>
     <xacro:kinect_camera prefix="camera" robot_namespace="$(arg robot_namespace)">
