Commit message: add support for mot tracker

File: husky_description/urdf/accessories/kinect_camera.urdf.xacro (robot description, xacro)
@@ -77,7 +77,7 @@
       <sensor type="depth" name="${prefix}">
         <always_on>true</always_on>
-        <update_rate>20.0</update_rate>
+        <update_rate>10.0</update_rate>
         <camera>
-          <horizontal_fov>${60.0*M_PI/180.0}</horizontal_fov>
+          <horizontal_fov>${70.0*M_PI/180.0}</horizontal_fov>
           <image>
             <format>R8G8B8</format>
@@ -107,5 +107,5 @@
           <distortion_t2>0.0</distortion_t2>
           <pointCloudCutoff>0.4</pointCloudCutoff>
-          <pointCloudCutoffMax>5.0</pointCloudCutoffMax>
+          <pointCloudCutoffMax>6.0</pointCloudCutoffMax>
           <robotNamespace>${robot_namespace}</robotNamespace>
         </plugin>

File: husky_description/urdf/accessories/sensor_arch.urdf.xacro (robot description, xacro)
@@ -6,10 +6,10 @@
              <origin xyz="0 0 0" rpy="0 0 0"/>
              <visual>
-		<origin xyz="0 0 -0.27" rpy="0 0 0"/>
+		<origin xyz="0 0 -0.40" rpy="0 0 0"/>
                  <!--geometry>
                      <mesh filename="package://husky_description/meshes/accessories/${size}_mm_sensor_arch.dae" />
                  </geometry-->
 		  <geometry>
-		   <cylinder radius="0.05" length="0.48"/>
+		   <cylinder radius="0.05" length="0.73"/>
 		  </geometry>
 	       	<material name="black"/>

File: husky_description/urdf/decorations.urdf.xacro (robot description, xacro)
@@ -161,4 +161,12 @@
             </geometry>
           </collision>
+        <inertial>
+          <origin xyz="0 0 0" rpy="0 0 0" />
+          <mass value="0.1" />
+          <inertia
+            ixx="0.0" ixy="0.0" ixz="0.0"
+            iyy="0.0" iyz="0.0"
+            izz="0.0" />
+        </inertial>
         </link>
         <!-- Attach top plate -->

File: husky_description/urdf/husky.urdf.xacro (robot description, xacro)
@@ -127,5 +127,5 @@
   <xacro:if value="$(arg kinect_enabled)">
     <xacro:sensor_arch prefix="" parent="top_plate_link">
-      <origin xyz="0 0 0.51" rpy="0 0 0"/>
+      <origin xyz="0 0 0.75" rpy="0 0 0"/>
     </xacro:sensor_arch>
     <xacro:kinect_camera prefix="camera" robot_namespace="$(arg robot_namespace)">
